File: rpcube.kicad_pcb (KiCad board)
At the start: 4 copper layers, 16.5 x 16.5 mm, 90 parts, among them J1 Conn_01x01_Female, J10 Conn_01x01_Female, J11 Conn_01x01_Female, J12 Conn_01x01_Female, J13 Conn_01x01_Female, J14 Conn_01x01_Female, J15 Conn_01x01_Female, J16 Conn_01x01_Female, J17 Conn_01x01_Female, J18 Conn_01x01_Female, J19 Conn_01x01_Female, J2 Conn_01x01_Female, J20 Conn_01x01_Female, J21 Conn_01x01_Female, J22 Conn_01x01_Female, J23 Conn_01x01_Female, J24 Conn_01x01_Female, J25 Conn_01x01_Female, J26 Conn_01x01_Female, J27 Conn_01x01_Female, J28 Conn_01x01_Female, J29 Conn_01x01_Female, J3 Conn_01x01_Female, J30 Conn_01x01_Female, J31 Conn_01x01_Female, J32 Conn_01x01_Female, J33 Conn_01x01_Female, J34 Conn_01x01_Female, J35 Conn_01x01_Female, J36 Conn_01x01_Female, J37 Conn_01x01_Female, J38 Conn_01x01_Female, J39 Conn_01x01_Female, J4 Conn_01x01_Female, J40 Conn_01x01_Female, J41 Conn_01x01_Female, J42 Conn_01x01_Female, J43 Conn_01x01_Female, J44 Conn_01x01_Female, J45 Conn_01x01_Female, J46 Conn_01x01_Female, J47 Conn_01x01_Female, J48 Conn_01x01_Female, J49 Conn_01x01_Female, J5 Conn_01x01_Female, J50 Conn_01x01_Female, J51 Conn_01x01_Female, J52 Conn_01x01_Female, J53 Conn_01x01_Female, J54 Conn_01x01_Female, J55 Conn_01x01_Female, J56 Conn_01x01_Female, J57 Conn_01x01_Female, J58 Conn_01x01_Female, J59 Conn_01x01_Female, J6 Conn_01x01_Female, J60 Conn_01x01_Female, J61 Conn_01x01_Female, J62 Conn_01x01_Female, J63 Conn_01x01_Female, J64 Conn_01x01_Female, J7 Conn_01x01_Female, J8 Conn_01x01_Female, J9 Conn_01x01_Female, U1 MIC5205-3.3YM5, U2 W25Q16JVUXIQ_TR, U3 RP2040, Y1 ECS-120-12-36-AGN-TR3

Commit message: minor changes
Parts:
- moved J48 0.38 mm to (81.3, 74.7)
Other:
- board text added: "1"
- board text added: "2"
- board text added: "3"
- board text added: "4"
- board text added: "5"
- board text added: "6"
- board text added: "7"
- board text added: "8"
- board text added: "A"
- board text added: "B"
- board text added: "C"
- board text added: "D"
- board text added: "E"
- board text added: "F"
- board text added: "G"
- board text added: "H"
Changed lines of the file:
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@@
   )
   (footprint "BGA_PAD:BGA_PAD" (layer "B.Cu")
-    (at 81.661 74.676 180)
+    (at 81.28 74.676 180)
     (property "Sheetfile" "rpcube.kicad_sch")
     (property "Sheetname" "")
@@
   )
   (gr_rect (start 76.073 59.309) (end 92.583 75.819) (layer "Edge.Cuts") (width 0.2) (fill none))
+  (gr_text "4" (at 85.344 58.42) (layer "B.SilkS")
+    (effects (font (size 1 1) (thickness 0.15)) (justify mirror))
+  )
+  (gr_text "G" (at 93.218 72.771) (layer "B.SilkS")
+    (effects (font (size 1 1) (thickness 0.15)) (justify mirror))
+  )
+  (gr_text "8" (at 77.216 58.42) (layer "B.SilkS")
+    (effects (font (size 1 1) (thickness 0.15)) (justify mirror))
+  )
+  (gr_text "5" (at 83.185 58.42) (layer "B.SilkS")
+    (effects (font (size 1 1) (thickness 0.15)) (justify mirror))
+  )
+  (gr_text "3" (at 87.376 58.42) (layer "B.SilkS")
+    (effects (font (size 1 1) (thickness 0.15)) (justify mirror))
+  )
+  (gr_text "1" (at 91.567 58.42) (layer "B.SilkS")
+    (effects (font (size 1 1) (thickness 0.15)) (justify mirror))
+  )
+  (gr_text "C" (at 93.218 64.643) (layer "B.SilkS")
+    (effects (font (size 1 1) (thickness 0.15)) (justify mirror))
+  )
+  (gr_text "B" (at 93.218 62.611) (layer "B.SilkS")
+    (effects (font (size 1 1) (thickness 0.15)) (justify mirror))
+  )
+  (gr_text "F" (at 93.218 70.739) (layer "B.SilkS")
+    (effects (font (size 1 1) (thickness 0.15)) (justify mirror))
+  )
+  (gr_text "A" (at 93.218 60.452) (layer "B.SilkS")
+    (effects (font (size 1 1) (thickness 0.15)) (justify mirror))
+  )
+  (gr_text "D" (at 93.218 66.675) (layer "B.SilkS")
+    (effects (font (size 1 1) (thickness 0.15)) (justify mirror))
+  )
+  (gr_text "7" (at 79.375 58.42) (layer "B.SilkS")
+    (effects (font (size 1 1) (thickness 0.15)) (justify mirror))
+  )
+  (gr_text "6" (at 81.28 58.42) (layer "B.SilkS")
+    (effects (font (size 1 1) (thickness 0.15)) (justify mirror))
+  )
+  (gr_text "E" (at 93.218 68.707) (layer "B.SilkS")
+    (effects (font (size 1 1) (thickness 0.15)) (justify mirror))
+  )
+  (gr_text "2" (at 89.408 58.42) (layer "B.SilkS")
+    (effects (font (size 1 1) (thickness 0.15)) (justify mirror))
+  )
+  (gr_text "H" (at 93.218 74.803) (layer "B.SilkS")
+    (effects (font (size 1 1) (thickness 0.15)) (justify mirror))
+  )
   (dimension (type aligned) (layer "User.1")
-    (pts (xy 76.073 75.819) (xy 92.583 75.819))
+    (pts (xy 76.073 77.089001) (xy 92.583 77.089001))
     (height 3.174999)
-    (gr_text "16.5100 mm" (at 84.328 77.843999) (layer "User.1")
+    (gr_text "16.5100 mm" (at 84.328 79.114) (layer "User.1")
       (effects (font (size 1 1) (thickness 0.15)))
     )
@@
   (segment (start 78.233562 75.0925) (end 78.8315 75.0925) (width 0.127) (layer "B.Cu") (net 25))
   (segment (start 78.8315 75.0925) (end 79.248 74.676) (width 0.127) (layer "B.Cu") (net 25))
-  (segment (start 79.248 74.676) (end 79.60015 75.02815) (width 0.127) (layer "F.Cu") (net 26))
-  (segment (start 83.055 71.605776) (end 82.431276 72.2295) (width 0.127) (layer "F.Cu") (net 26))
-  (segment (start 79.248 73.152) (end 79.248 74.676) (width 0.127) (layer "F.Cu") (net 26))
-  (segment (start 82.431276 72.2295) (end 81.348552 72.2295) (width 0.127) (layer "F.Cu") (net 26))
-  (segment (start 81.348552 72.2295) (end 81.347052 72.228) (width 0.127) (layer "F.Cu") (net 26))
-  (segment (start 81.347052 72.228) (end 80.172 72.228) (width 0.127) (layer "F.Cu") (net 26))
-  (segment (start 83.055 70.8745) (end 83.055 71.605776) (width 0.127) (layer "F.Cu") (net 26))
-  (segment (start 80.172 72.228) (end 79.248 73.152) (width 0.127) (layer "F.Cu") (net 26))
-  (segment (start 79.60015 75.02815) (end 80.289583 75.02815) (width 0.127) (layer "F.Cu") (net 26))
-  (via (at 80.289583 75.02815) (size 0.8) (drill 0.4) (layers "F.Cu" "B.Cu") (net 26))
-  (segment (start 80.641733 74.676) (end 81.661 74.676) (width 0.127) (layer "B.Cu") (net 26))
-  (segment (start 80.289583 75.02815) (end 80.641733 74.676) (width 0.127) (layer "B.Cu") (net 26))
+  (segment (start 81.347052 72.228) (end 81.348552 72.2295) (width 0.127) (layer "F.Cu") (net 26))
+  (segment (start 83.055 71.605776) (end 83.055 70.8745) (width 0.127) (layer "F.Cu") (net 26))
+  (segment (start 79.248 74.676) (end 79.248 73.152) (width 0.127) (layer "F.Cu") (net 26))
+  (segment (start 80.172 72.228) (end 81.347052 72.228) (width 0.127) (layer "F.Cu") (net 26))
+  (segment (start 80.373498 75.02815) (end 79.60015 75.02815) (width 0.127) (layer "F.Cu") (net 26))
+  (segment (start 82.431276 72.2295) (end 83.055 71.605776) (width 0.127) (layer "F.Cu") (net 26))
+  (segment (start 79.248 73.152) (end 80.172 72.228) (width 0.127) (layer "F.Cu") (net 26))
+  (segment (start 79.60015 75.02815) (end 79.248 74.676) (width 0.127) (layer "F.Cu") (net 26))
+  (segment (start 81.348552 72.2295) (end 82.431276 72.2295) (width 0.127) (layer "F.Cu") (net 26))
+  (via (at 80.373498 75.02815) (size 0.8) (drill 0.4) (layers "F.Cu" "B.Cu") (net 26))
+  (segment (start 80.373498 75.02815) (end 80.725648 74.676) (width 0.127) (layer "B.Cu") (net 26))
+  (segment (start 80.725648 74.676) (end 81.661 74.676) (width 0.127) (layer "B.Cu") (net 26))
   (segment (start 86.655 71.355356) (end 86.655 70.8745) (width 0.127) (layer "F.Cu") (net 27))
   (segment (start 88.650875 72.328896) (end 88.584896 72.328896) (width 0.127) (layer "F.Cu") (net 27))
