File: rpcube.kicad_pcb (KiCad board)
At the start: 4 copper layers, 16.5 x 16.5 mm, 90 parts, among them J1 Conn_01x01_Female, J10 Conn_01x01_Female, J11 Conn_01x01_Female, J12 Conn_01x01_Female, J13 Conn_01x01_Female, J14 Conn_01x01_Female, J15 Conn_01x01_Female, J16 Conn_01x01_Female, J17 Conn_01x01_Female, J18 Conn_01x01_Female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

Commit message: added more images
Other:
- board text added: "PCB3D_BR_rpcube"
- board text added: "PCB3D_TL_rpcube"
